Commit message: Add files via upload

File: hand__description/urdf/hand_.xacro (robot description, xacro)
@@ -206,7 +206,7 @@
 <link name="i_pip_pitch_link_v4_1">
   <inertial>
-    <origin xyz="0.0010000000000000044 0.001096507521878223 0.018000000026317478" rpy="0 0 0"/>
-    <mass value="0.0314105238001653"/>
-    <inertia ixx="7e-06" iyy="8e-06" izz="2e-06" ixy="-0.0" iyz="-0.0" ixz="0.0"/>
+    <origin xyz="0.0010000000000000044 -4.163336342344337e-17 0.0179999999696749" rpy="0 0 0"/>
+    <mass value="0.005240569245269249"/>
+    <inertia ixx="2e-06" iyy="2e-06" izz="0.0" ixy="-0.0" iyz="0.0" ixz="-0.0"/>
   </inertial>
   <visual>
@@ -246,7 +246,7 @@
 <link name="i_dip_link_v2_1">
   <inertial>
-    <origin xyz="0.0010000228538777876 0.000633326000430515 0.005499983676315989" rpy="0 0 0"/>
-    <mass value="0.0165936992661325"/>
-    <inertia ixx="1e-06" iyy="1e-06" izz="1e-06" ixy="0.0" iyz="-0.0" ixz="0.0"/>
+    <origin xyz="0.0010000000000000078 -7.112366251504909e-17 0.005499999970720593" rpy="0 0 0"/>
+    <mass value="0.005240569245269249"/>
+    <inertia ixx="0.0" iyy="0.0" izz="0.0" ixy="0.0" iyz="-0.0" ixz="0.0"/>
   </inertial>
   <visual>
@@ -366,7 +366,7 @@
 <link name="m_pip_pitch_link_v2_1">
   <inertial>
-    <origin xyz="-0.0031359988745470087 -0.00039822543823583335 0.018383211430427746" rpy="0 0 0"/>
-    <mass value="0.03753911672457911"/>
-    <inertia ixx="7e-06" iyy="1.1e-05" izz="6e-06" ixy="-0.0" iyz="0.0" ixz="0.0"/>
+    <origin xyz="-0.010824012750029453 0.0007615456375304318 0.018123960084147656" rpy="0 0 0"/>
+    <mass value="0.11604898173137333"/>
+    <inertia ixx="2.2e-05" iyy="7.8e-05" izz="6.1e-05" ixy="0.0" iyz="0.0" ixz="0.0"/>
   </inertial>
   <visual>
@@ -406,7 +406,7 @@
 <link name="m_dip_link_v2_1">
   <inertial>
-    <origin xyz="-0.0014999771461222094 0.0005852527718479845 0.005505359071886956" rpy="0 0 0"/>
-    <mass value="0.0165936992661325"/>
-    <inertia ixx="1e-06" iyy="1e-06" izz="1e-06" ixy="0.0" iyz="0.0" ixz="0.0"/>
+    <origin xyz="-0.0014999999999999911 -4.804925566282911e-05 0.005499848623846337" rpy="0 0 0"/>
+    <mass value="0.005240569245269249"/>
+    <inertia ixx="0.0" iyy="0.0" izz="0.0" ixy="0.0" iyz="0.0" ixz="-0.0"/>
   </inertial>
   <visual>
@@ -526,7 +526,7 @@
 <link name="r_pip_pitch_link_v2_1">
   <inertial>
-    <origin xyz="-0.001500000000000029 0.00109650752187823 0.017999999914078108" rpy="0 0 0"/>
-    <mass value="0.0314105238001653"/>
-    <inertia ixx="7e-06" iyy="8e-06" izz="2e-06" ixy="0.0" iyz="0.0" ixz="-0.0"/>
+    <origin xyz="-0.001500000000000029 -3.469446951953614e-17 0.01799999997072063" rpy="0 0 0"/>
+    <mass value="0.005240569245269249"/>
+    <inertia ixx="2e-06" iyy="2e-06" izz="0.0" ixy="0.0" iyz="0.0" ixz="-0.0"/>
   </inertial>
   <visual>
@@ -566,7 +566,7 @@
 <link name="r_dip_link_v2_1">
   <inertial>
-    <origin xyz="0.0010000228538776974 0.0006333260004305185 0.005499983676316045" rpy="0 0 0"/>
-    <mass value="0.0165936992661325"/>
-    <inertia ixx="1e-06" iyy="1e-06" izz="1e-06" ixy="0.0" iyz="-0.0" ixz="0.0"/>
+    <origin xyz="0.0009999999999999176 -7.112366251504909e-17 0.005499999970720648" rpy="0 0 0"/>
+    <mass value="0.005240569245269249"/>
+    <inertia ixx="0.0" iyy="0.0" izz="0.0" ixy="0.0" iyz="0.0" ixz="0.0"/>
   </inertial>
   <visual>
@@ -686,7 +686,7 @@
 <link name="s_pip_pitch_link_v2_1">
   <inertial>
-    <origin xyz="0.0010000000000000009 0.0010965075218782126 0.018000000026317423" rpy="0 0 0"/>
-    <mass value="0.0314105238001653"/>
-    <inertia ixx="7e-06" iyy="8e-06" izz="2e-06" ixy="0.0" iyz="-0.0" ixz="-0.0"/>
+    <origin xyz="0.0010000000000000078 -5.204170427930421e-17 0.017999999969674843" rpy="0 0 0"/>
+    <mass value="0.005240569245269249"/>
+    <inertia ixx="2e-06" iyy="2e-06" izz="0.0" ixy="0.0" iyz="0.0" ixz="-0.0"/>
   </inertial>
   <visual>
@@ -726,7 +726,7 @@
 <link name="s_dip_link_v2_1">
   <inertial>
-    <origin xyz="0.0038505897470794623 -0.00013446931523418415 0.0053744656124536105" rpy="0 0 0"/>
-    <mass value="0.01838422914819263"/>
-    <inertia ixx="1e-06" iyy="4e-06" izz="3e-06" ixy="0.0" iyz="-0.0" ixz="0.0"/>
+    <origin xyz="0.02728839732396658 0.00047118040829075003 0.005456277585069891" rpy="0 0 0"/>
+    <mass value="0.05228120754232652"/>
+    <inertia ixx="3e-06" iyy="3.1e-05" izz="3e-05" ixy="-0.0" iyz="-0.0" ixz="0.0"/>
   </inertial>
   <visual>
